Commit message: 11/20

File: src/vis_lecture/xacro/rollerWalker_gazebo.xacro (robot description, xacro)
@@ -123,5 +123,5 @@
         </joint>
         <!-- ジョイント2のトランスミッション -->
-        <transmission name="joint_2_${leg_posi}_trans" type="SimpleTransmission">
+        <transmission name="joint_2_${leg_posi}_trans" >
             <type>transmission_interface/SimpleTransmission</type>
             <actuator name="$joint_2_${leg_posi}_motor">
@@ -198,5 +198,5 @@
         </joint>
         <!-- ジョイント3のトランスミッション -->
-        <transmission name="joint_3_${leg_posi}_trans" type="SimpleTransmission">
+        <transmission name="joint_3_${leg_posi}_trans" >
             <type>transmission_interface/SimpleTransmission</type>
             <actuator name="$joint_3_${leg_posi}_motor">
@@ -272,5 +272,5 @@
         </joint>
         <!-- ジョイント3のトランスミッション -->
-        <transmission name="joint_4_${leg_posi}_trans" type="SimpleTransmission">
+        <transmission name="joint_4_${leg_posi}_trans" >
             <type>transmission_interface/SimpleTransmission</type>
             <actuator name="$joint_4_${leg_posi}_motor">
@@ -346,5 +346,5 @@
         </joint>
         <!-- ジョイント3のトランスミッション -->
-        <transmission name="wheel_trans" type="SimpleTransmission">
+        <transmission name="wheel_trans" >
             <type>transmission_interface/SimpleTransmission</type>
             <actuator name="$wheel_motor">
@@ -420,8 +420,8 @@
         <origin xyz="${body_length/2 - joint_1_radius/2} ${body_width/2 - joint_1_radius/2} 0.0" rpy="0 0 0"/>
         <dynamics damping="${body_to_joint_1_damping}"/>
-        <limit lower="0.1" upper="3" effort="0" velocity="0"/>
+        <limit lower="0.2" upper="3" effort="0" velocity="0"/>
     </joint>
     <!-- ジョイント1_LFトランスミッション設定 -->
-    <transmission name="joint_1_lf_trans" type="SimpleTransmission">
+    <transmission name="joint_1_lf_trans" >
         <type>transmission_interface/SimpleTransmission</type>
         <actuator name="$joint_1_lf_motor">
@@ -462,8 +462,8 @@
         <origin xyz="${-(body_length/2 - joint_1_radius/2)} ${body_width/2 - joint_1_radius/2} 0.0" rpy="0 0 0"/>
         <dynamics damping="${body_to_joint_1_damping}"/>
-        <limit lower="0.1" upper="3" effort="0" velocity="0"/>
+        <limit lower="0.2" upper="3" effort="0" velocity="0"/>
     </joint>
     <!-- ジョイント1_LRトランスミッション設定 -->
-    <transmission name="joint_1_lr_trans" type="SimpleTransmission">
+    <transmission name="joint_1_lr_trans" >
         <type>transmission_interface/SimpleTransmission</type>
         <actuator name="$joint_1_lr_motor">
@@ -504,8 +504,8 @@
         <origin xyz="${-(body_length/2 - joint_1_radius/2)} ${-(body_width/2 - joint_1_radius/2)} 0.0" rpy="0 0 0"/>
         <dynamics damping="${body_to_joint_1_damping}"/>
-        <limit lower="-3" upper="-0.1" effort="0" velocity="0"/>
+        <limit lower="-3" upper="-0.2" effort="0" velocity="0"/>
     </joint>
     <!-- ジョイント1_RRトランスミッション設定 -->
-    <transmission name="joint_1_rr_trans" type="SimpleTransmission">
+    <transmission name="joint_1_rr_trans" >
         <type>transmission_interface/SimpleTransmission</type>
         <actuator name="$joint_1_rr_motor">
@@ -546,8 +546,8 @@
         <origin xyz="${body_length/2 - joint_1_radius/2} ${-(body_width/2 - joint_1_radius/2)} 0.0" rpy="0 0 0"/>
         <dynamics damping="${body_to_joint_1_damping}"/>
-        <limit lower="-3" upper="-0.1" effort="0" velocity="0"/>
+        <limit lower="-3" upper="-0.2" effort="0" velocity="0"/>
     </joint>
     <!-- ジョイント1_RFトランスミッション設定 -->
-    <transmission name="joint_1_rf_trans" type="SimpleTransmission">
+    <transmission name="joint_1_rf_trans" >
         <type>transmission_interface/SimpleTransmission</type>
         <actuator name="$joint_1_rf_motor">

Commit message: change joint_limit

File: src/vis_lecture/xacro/rollerWalker_gazebo.xacro (robot description, xacro)
@@ -120,5 +120,5 @@
             <origin rpy="1.57070 0 0" xyz="0 0 0"/>
             <dynamics damping="${joint_1_to_joint_2_damping}"/>
-            <limit lower="-1.5" upper="1.5" effort="0" velocity="0"/>
+            <limit lower="-1.5" upper="1.5" effort="100" velocity="100"/>
         </joint>
         <!-- ジョイント2のトランスミッション -->
@@ -195,5 +195,5 @@
             <origin rpy="1.57070 0 0" xyz="${link_2_x} 0 0"/>
             <dynamics damping="${link_2_to_joint_3_damping}"/>
-            <limit lower="-2.0" upper="1.5" effort="0" velocity="0"/>
+            <limit lower="-2.0" upper="1.5" effort="100" velocity="100"/>
         </joint>
         <!-- ジョイント3のトランスミッション -->
@@ -269,5 +269,5 @@
             <origin rpy="1.57070 0 0" xyz="${link_3_x} 0 0"/>
             <dynamics damping="${link_3_to_joint_4_damping}"/>
-            <limit lower="-2.0" upper="1.5" effort="0" velocity="0"/>
+            <limit lower="-2.0" upper="1.5" effort="100" velocity="100"/>
         </joint>
         <!-- ジョイント3のトランスミッション -->
@@ -420,5 +420,5 @@
         <origin xyz="${body_length/2 - joint_1_radius/2} ${body_width/2 - joint_1_radius/2} 0.0" rpy="0 0 0"/>
         <dynamics damping="${body_to_joint_1_damping}"/>
-        <limit lower="0.2" upper="3" effort="0" velocity="0"/>
+        <limit lower="0.2" upper="3" effort="100" velocity="100"/>
     </joint>
     <!-- ジョイント1_LFトランスミッション設定 -->
@@ -462,5 +462,5 @@
         <origin xyz="${-(body_length/2 - joint_1_radius/2)} ${body_width/2 - joint_1_radius/2} 0.0" rpy="0 0 0"/>
         <dynamics damping="${body_to_joint_1_damping}"/>
-        <limit lower="0.2" upper="3" effort="0" velocity="0"/>
+        <limit lower="0.2" upper="3" effort="100" velocity="100"/>
     </joint>
     <!-- ジョイント1_LRトランスミッション設定 -->
@@ -504,5 +504,5 @@
         <origin xyz="${-(body_length/2 - joint_1_radius/2)} ${-(body_width/2 - joint_1_radius/2)} 0.0" rpy="0 0 0"/>
         <dynamics damping="${body_to_joint_1_damping}"/>
-        <limit lower="-3" upper="-0.2" effort="0" velocity="0"/>
+        <limit lower="-3" upper="-0.2" effort="100" velocity="100"/>
     </joint>
     <!-- ジョイント1_RRトランスミッション設定 -->
@@ -546,5 +546,5 @@
         <origin xyz="${body_length/2 - joint_1_radius/2} ${-(body_width/2 - joint_1_radius/2)} 0.0" rpy="0 0 0"/>
         <dynamics damping="${body_to_joint_1_damping}"/>
-        <limit lower="-3" upper="-0.2" effort="0" velocity="0"/>
+        <limit lower="-3" upper="-0.2" effort="100" velocity="100"/>
     </joint>
     <!-- ジョイント1_RFトランスミッション設定 -->
